File: Kicad/PAMI_TEAM_SCRAT_FINAL/PAMI_TEAM_SCRAT_FINAL.kicad_sch (KiCad schematic)
At the start: 48 parts, among them J1 ALIM, J2 TOF, J3 IR, J4 M1, J5 M2, J6 XL320, SW1 BTN1, SW2 BTN2, SW3 BTN3, U3 WE-DC-DC-5V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

Commit message: update pcb
Other:
- moved on the sheet: C1, C11, C12, C13, C14, C15, C16, C17, C18, C2, C21, C22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

Commit message: pcb termine
Parts:
- added D2, D3: LED, LED_SMD:LED_0603_1608Metric, symbol Device:LED
- added R10: 3k3, Resistor_SMD:R_0603_1608Metric, symbol Device:R
- added R11: 5k8, Resistor_SMD:R_0603_1608Metric, symbol Device:R
- D1: MPN (none) -> 150060RS55040
- R8: value 510 -> 1k6
- SW1, SW2, SW3: footprint Button_Switch_SMD:Panasonic_EVQPUJ_EVQPUA -> Button_Switch_SMD:SW_SPST_PTS645Sx43SMTR92
- U3: value WE-DC-DC-5V -> 173010578; MPN (none) -> 173010578
- renumbered D2 to D4, D3 to D5, D4 to D6, D5 to D7, D6 to D8, D7 to D9
Connections:
- net +3.3V: no longer D4.3 (VDD), D5.3 (VDD), D6.3 (VDD), D7.3 (VDD), D8.3 (VDD), D9.3 (VDD)
- net +7.5V: now also R11.1
- net A_ENC1: now also J5.3 (Pin_3); no longer J4.3 (Pin_3)
- net A_ENC2: now also J5.4 (Pin_4); no longer J4.4 (Pin_4)
- net A_O1: now also J5.1 (Pin_1); no longer J4.1 (Pin_1)
- net A_O2: now also J5.6 (Pin_6); no longer J4.6 (Pin_6)
- net B_ENC1: now also J4.3 (Pin_3); no longer J5.3 (Pin_3)
- net B_ENC2: now also J4.4 (Pin_4); no longer J5.4 (Pin_4)
- net B_O1: now also J4.1 (Pin_1); no longer J5.1 (Pin_1)
- net B_O2: now also J4.6 (Pin_6); no longer J5.6 (Pin_6)
- net GND: now also D2.1 (K), D3.1 (K)
- net +5V: now reaches C11.1, U3.3 (OUT), U4.1 (IN)
- net +5V: now also D4.3 (VDD), D5.3 (VDD), D6.3 (VDD), D7.3 (VDD), D8.3 (VDD), D9.3 (VDD), R10.1
- new net: D3.2 (A), R11.2
- new net: D2.2 (A), R10.2
Other:
- note added: "1.7V @ 1mA"
- moved on the sheet: C1, C11, C12, C13, C14, C15, C16, C17, C18, C2, C21, C22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
